File: BBCWinchesterPro.kicad_pcb (KiCad board)
At the start: 2 copper layers, 97.5 x 165 mm, 37 parts, among them J1 Conn_02x17_Odd_Even, J2 Conn_01x04_Male, J3 Conn_01x02_Male, J4 Conn_02x20_Odd_Even, J5 Conn_02x20_Odd_Even, J6 Conn_02x20_Odd_Even, P1 CONN_01X02, P2 CONN_01x03, U1 74LS02, U2 74LS139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

Commit message: Add ATTiny code and remove license from silkscreen
Other:
- board text added: "https://github.com/marrold/BBCWinchesterPro v0.2"
- board text removed: "https://github.com/marrold/BBCWinchesterPro Licensed under CC BY-NC-SA v0.1"
